Commit message: push it

File: robotic_arm.urdf (robot description, URDF)
Before this commit: robot measured_robotic_hand_arm, 9 links, 8 joints
Links:
- added link mobile_base_link, mass 2.0; collision box size=0.22 0.18 0.18; visual box size=0.22 0.18 0.18
Joints:
- added joint mobile_base_to_arm_base: type fixed, parent mobile_base_link, child base_link, origin xyz=0 0 0.18 rpy=0 0 0

Commit message: update urdf!!

File: robotic_arm.urdf (robot description, URDF)
Before this commit: robot measured_robotic_hand_arm, 10 links, 9 joints
Joints:
- joint mobile_base_to_arm_base: origin xyz=0 0 0.18 rpy=0 0 0 -> xyz=0 0 0.15 rpy=0 0 0
